Commit message: Imported upstream version '0.0.4' of 'upstream'

File: asus_description/urdf/asus/asus.xacro (robot description, xacro)
@@ -2,135 +2,8 @@
 <robot name="asus_sensor" xmlns:xacro="http://www.ros.org/wiki/xacro">
     <xacro:macro name="asus_sensor" params="prefix name parent cam_px cam_py cam_pz cam_or cam_op cam_oy">
-        <xacro:property name="M_SCALE" value="0.001"/>
-        <xacro:property name="M_PI" value="3.141592"/>
-        <link name="${name}_link">
-            <visual>
-                <geometry>
-                    <mesh filename="package://turtlebot_description/meshes/sensors/asus_xtion_pro_live.dae" scale="${M_SCALE} ${M_SCALE} ${M_SCALE}"/>
-                </geometry>
-                <origin xyz="-0.01 0 0" rpy="${-M_PI/2} -${M_PI} ${-M_PI/2}"/>
-            </visual>
-            <collision>
-                <geometry>
-                    <box size="0.0730 0.2760 0.0720"/>
-                </geometry>
-                <contact_coefficients mu="0" kp="1000.0" kd="1.0"/>
-            </collision>
-            <inertial>
-                <mass value="0.170" />
-                <origin xyz="0 0 0" />
-                <inertia ixx="0.001152600" ixy="0.0" ixz="0.0" iyy="0.000148934" iyz="0.0" izz="0.001154654" />
-            </inertial>
-        </link>
-        <joint name="${name}_joint" type="fixed">
-            <parent link="${parent}"/>
-            <child link="${name}_link"/>
-            <origin xyz="${cam_px} ${cam_py} ${cam_pz}" rpy="${cam_or} ${cam_op} ${cam_oy}"/>
-        </joint>
-        <link name="${name}_rgb_optical_frame"/>
-        <joint name="${name}_rgb_joint" type="fixed">
-            <parent link="${name}_link"/>
-            <child link="${name}_rgb_optical_frame"/>
-            <origin xyz="0 0.0125 0.016" rpy="-1.57 0 -1.57"/>
-        </joint>
-        <link name="${name}_depth_optical_frame"/>
-        <joint name="${name}_depth_joint" type="fixed">
-            <parent link="${name}_link"/>
-            <child link="${name}_depth_optical_frame"/>
-            <origin xyz="0 -0.0125 0.016" rpy="-1.57 0 -1.57"/>
-        </joint>
-        <!-- Not sure why in a macro arguments cannot be passed to an
-        associated .gazebo.xacro file... -->
-        <!-- See https://github.com/turtlebot/turtlebot and there
-        turtlebot_description/urdf/turtlebot_gazebo.urdf.xacro -->
-        <gazebo reference="${name}_link">
-            <sensor name="${name}_sensor" type="depth">
-                <always_on>true</always_on>
-                <update_rate>20.0</update_rate>
-                <camera>
-                    <horizontal_fov>${60.0*M_PI/180.0}</horizontal_fov>
-                    <image>
-                        <width>640</width>
-                        <height>480</height>
-                        <format>B8G8R8</format>
-                    </image>
-                    <clip>
-                        <near>0.05</near>
-                        <far>8.0</far>
-                    </clip>
-                    <noise>
-                        <!-- Noise is sampled independently per pixel on each frame.
-                        That pixel's noise value is added to each of its color
-                        channels, which at that point lie in the range [0,1]. -->
-                        <type>gaussian</type>
-                        <mean>0.0</mean>
-                        <stddev>0.001</stddev>
-                    </noise>
-                </camera>
-                <plugin name="${name}_sensor_controller"
-                        filename="libgazebo_ros_openni_kinect.so">
-                    <cameraName>${name}</cameraName>
-                    <alwaysOn>true</alwaysOn>
-                    <updateRate>10.0</updateRate>
-                    <imageTopicName>rgb/image_raw</imageTopicName>
-                    <depthImageTopicName>depth/image_raw</depthImageTopicName>
-                    <pointCloudTopicName>depth/points</pointCloudTopicName>
-                    <cameraInfoTopicName>rgb/camera_info</cameraInfoTopicName>
-                    <depthImageCameraInfoTopicName>depth/camera_info</depthImageCameraInfoTopicName>
-                    <frameName>${name}_depth_optical_frame</frameName>
-                    <pointCloudCutoff>0.4</pointCloudCutoff>
-                    <pointCloudCutoffMax>8.0</pointCloudCutoffMax>
-                    <baseline>0.1</baseline>
-                    <distortion_k1>0.0</distortion_k1>
-                    <distortion_k2>0.0</distortion_k2>
-                    <distortion_k3>0.0</distortion_k3>
-                    <distortion_t1>0.0</distortion_t1>
-                    <distortion_t2>0.0</distortion_t2>
-                    <robotNamespace>${prefix}</robotNamespace>
-                </plugin>
-            </sensor>
-        </gazebo>
-        <gazebo reference="${name}_link">
-            <sensor name="${name}_camera" type="camera">
-                <always_on>true</always_on>
-                <update_rate>30.0</update_rate>
-                <camera name="${name}_camera">
-                    <horizontal_fov>${60.0*M_PI/180.0}</horizontal_fov>
-                    <image>
-                        <width>1280</width>
-                        <height>1024</height>
-                        <format>R8G8B8</format>
-                    </image>
-                    <clip>
-                        <near>0.02</near>
-                        <far>10.0</far>
-                    </clip>
-                    <noise>
-                        <!-- Noise is sampled independently per pixel on each frame.
-                        That pixel's noise value is added to each of its color
-                        channels, which at that point lie in the range [0,1]. -->
-                        <type>gaussian</type>
-                        <mean>0.0</mean>
-                        <stddev>0.007</stddev>
-                    </noise>
-                </camera>
-                <plugin name="${name}_camera_controller"
-                        filename="libgazebo_ros_camera.so">
-                    <alwaysOn>true</alwaysOn>
-                    <update_rate>30.0</update_rate>
-                    <cameraName>${name}</cameraName>
-                    <imageTopicName>hd/image_color_rect</imageTopicName>
-                    <cameraInfoTopicName>hd/camera_info</cameraInfoTopicName>
-                    <frameName>${name}_rgb_optical_frame</frameName>
-                    <baseline>0.1</baseline>
-                    <distortionK1>0.0</distortionK1>
-                    <distortionK2>0.0</distortionK2>
-                    <distortionK3>0.0</distortionK3>
-                    <distortionT1>0.0</distortionT1>
-                    <distortionT2>0.0</distortionT2>
-                    <robotNamespace>${prefix}</robotNamespace>
-                </plugin>
-            </sensor>
-        </gazebo>
+      <xacro:include filename="$(find asus_description)/urdf/asus/asus-no-gazebo.xacro"/>
+      <asus_sensor-ng  parent="${parent}" name="${name}" cam_px="${cam_px}" cam_py="${cam_py}" cam_pz="${cam_pz}" cam_or="${cam_or}" cam_op="${cam_op}" cam_oy="${cam_oy}"/>
+      <xacro:include filename="$(find asus_description)/urdf/asus/asus-gazebo.xacro"/>
+      <asus_sensor-g prefix="${prefix}" name="${name}"/>
     </xacro:macro>
 </robot>

File: kinect2_description/urdf/kinect2/kinect2.xacro (robot description, xacro)
@@ -2,133 +2,8 @@
 <robot name="kinect2_sensor" xmlns:xacro="http://www.ros.org/wiki/xacro">
     <xacro:macro name="kinect2_sensor" params="prefix name parent cam_px cam_py cam_pz cam_or cam_op cam_oy">
-        <link name="${name}_link">
-            <visual>
-                <geometry>
-                    <mesh filename="package://kinect2_description/meshes/sensors/kinect2.dae"/>
-                </geometry>
-                <origin xyz="0.02 0 0" rpy="0 0 3.141592"/>
-            </visual>
-            <collision>
-                <geometry>
-                    <box size=".1 .25 .06"/>
-                </geometry>
-                <contact_coefficients mu="0" kp="1000.0" kd="1.0"/>
-            </collision>
-            <inertial>
-                <mass value="1e-5" />
-                <origin xyz="0 0 0" rpy="0 0 0"/>
-                <inertia ixx="1e-6" ixy="0" ixz="0" iyy="1e-6" iyz="0" izz="1e-6" />
-            </inertial>
-        </link>
-        <joint name="${name}_joint" type="fixed">
-            <parent link="${parent}"/>
-            <child link="${name}_link"/>
-            <origin xyz="${cam_px} ${cam_py} ${cam_pz}" rpy="${cam_or} ${cam_op} ${cam_oy}"/>
-        </joint>
-        <link name="${name}_rgb_optical_frame"/>
-        <joint name="${name}_rgb_joint" type="fixed">
-            <parent link="${name}_link"/>
-            <child link="${name}_rgb_optical_frame"/>
-            <origin xyz="0 0.0125 0.016" rpy="-1.57 0 -1.57"/>
-        </joint>
-        <link name="${name}_depth_optical_frame"/>
-        <joint name="${name}_depth_joint" type="fixed">
-            <parent link="${name}_link"/>
-            <child link="${name}_depth_optical_frame"/>
-            <origin xyz="0 -0.0125 0.016" rpy="-1.57 0 -1.57"/>
-        </joint>
-        <!-- Not sure why in a macro arguments cannot be passed to an
-        associated .gazebo.xacro file... -->
-        <!-- See https://github.com/turtlebot/turtlebot and there
-        turtlebot_description/urdf/turtlebot_gazebo.urdf.xacro -->
-        <gazebo reference="${name}_link">
-            <sensor name="${name}_sensor" type="depth">
-                <always_on>true</always_on>
-                <update_rate>30.0</update_rate>
-                <camera>
-                    <horizontal_fov>${70.0*3.14/180.0}</horizontal_fov>
-                    <image>
-                        <width>512</width>
-                        <height>424</height>
-                        <format>L8</format>
-                    </image>
-                    <clip>
-                        <near>0.1</near>
-                        <far>8.0</far>
-                    </clip>
-                    <noise>
-                        <!-- Noise is sampled independently per pixel on each frame.
-                        That pixel's noise value is added to each of its color
-                        channels, which at that point lie in the range [0,1]. -->
-                        <type>gaussian</type>
-                        <mean>0.0</mean>
-                        <stddev>0.001</stddev>
-                    </noise>
-                </camera>
-                <plugin name="${name}_sensor_controller"
-                        filename="libgazebo_ros_openni_kinect.so">
-                    <cameraName>${name}</cameraName>
-                    <alwaysOn>true</alwaysOn>
-                    <updateRate>30.0</updateRate>
-                    <imageTopicName>sd/image_ir_rect</imageTopicName>
-                    <depthImageTopicName>sd/image_depth_rect</depthImageTopicName>
-                    <pointCloudTopicName>sd/points</pointCloudTopicName>
-                    <cameraInfoTopicName>sd/camera_info</cameraInfoTopicName>
-                    <!--<depthImageCameraInfoTopicName>depth/camera_info</depthImageCameraInfoTopicName>-->
-                    <frameName>${name}_depth_optical_frame</frameName>
-                    <pointCloudCutoff>0.5</pointCloudCutoff>
-                    <pointCloudCutoffMax>8.0</pointCloudCutoffMax>
-                    <baseline>0.1</baseline>
-                    <distortionK1>0.0</distortionK1>
-                    <distortionK2>0.0</distortionK2>
-                    <distortionK3>0.0</distortionK3>
-                    <distortionT1>0.0</distortionT1>
-                    <distortionT2>0.0</distortionT2>
-                    <robotNamespace>${prefix}</robotNamespace>
-                </plugin>
-            </sensor>
-        </gazebo>
-        <gazebo reference="${name}_link">
-            <sensor name="${name}_camera" type="camera">
-                <always_on>true</always_on>
-                <update_rate>30.0</update_rate>
-                <camera name="${name}_camera">
-                    <horizontal_fov>${84.1*3.14/180.0}</horizontal_fov>
-                    <image>
-                        <width>1920</width>
-                        <height>1080</height>
-                        <format>R8G8B8</format>
-                    </image>
-                    <clip>
-                        <near>0.02</near>
-                        <far>10.0</far>
-                    </clip>
-                    <noise>
-                        <!-- Noise is sampled independently per pixel on each frame.
-                        That pixel's noise value is added to each of its color
-                        channels, which at that point lie in the range [0,1]. -->
-                        <type>gaussian</type>
-                        <mean>0.0</mean>
-                        <stddev>0.007</stddev>
-                    </noise>
-                </camera>
-                <plugin name="${name}_camera_controller"
-                        filename="libgazebo_ros_camera.so">
-                    <alwaysOn>true</alwaysOn>
-                    <update_rate>30.0</update_rate>
-                    <cameraName>${name}</cameraName>
-                    <imageTopicName>hd/image_color_rect</imageTopicName>
-                    <cameraInfoTopicName>hd/camera_info</cameraInfoTopicName>
-                    <frameName>${name}_rgb_optical_frame</frameName>
-                    <baseline>0.1</baseline>
-                    <distortionK1>0.0</distortionK1>
-                    <distortionK2>0.0</distortionK2>
-                    <distortionK3>0.0</distortionK3>
-                    <distortionT1>0.0</distortionT1>
-                    <distortionT2>0.0</distortionT2>
-                    <robotNamespace>${prefix}</robotNamespace>
-                </plugin>
-            </sensor>
-        </gazebo>
+      <xacro:include filename="$(find kinect2_description)/urdf/kinect2/kinect2-no-gazebo.xacro"/>
+      <kinect2_sensor-ng parent="${parent}" name="${name}" cam_px="${cam_px}" cam_py="${cam_py}" cam_pz="${cam_pz}" cam_or="${cam_or}" cam_op="${cam_op}" cam_oy="${cam_oy}"/>
+      <xacro:include filename="$(find kinect2_description)/urdf/kinect2/kinect2-gazebo.xacro"/>
+      <kinect2_sensor-g prefix="${prefix}" name="${name}"/>
     </xacro:macro>
 </robot>
