Commit message: Imported upstream version '0.1.0' of 'upstream'

File: asus_description/urdf/asus/asus-no-gazebo.xacro (robot description, xacro)
@@ -7,5 +7,5 @@
             <visual>
                 <geometry>
-                    <mesh filename="package://turtlebot_description/meshes/sensors/asus_xtion_pro_live.dae" scale="${M_SCALE} ${M_SCALE} ${M_SCALE}"/>
+                    <mesh filename="package://asus_description/meshes/sensors/asus_xtion_pro_live.dae" scale="${M_SCALE} ${M_SCALE} ${M_SCALE}"/>
                 </geometry>
                 <origin xyz="-0.01 0 0" rpy="${-M_PI/2} -${M_PI} ${-M_PI/2}"/>

File: kinect2_description/urdf/kinect2/kinect2-gazebo.xacro (robot description, xacro)
@@ -2,4 +2,5 @@
 <robot name="kinect2_sensor-g" xmlns:xacro="http://www.ros.org/wiki/xacro">
     <xacro:macro name="kinect2_sensor-g" params="prefix name">
+        <xacro:property name="PI" value="3.14159265359" />
         <!-- See https://github.com/turtlebot/turtlebot and there
         turtlebot_description/urdf/turtlebot_gazebo.urdf.xacro -->
@@ -9,5 +10,5 @@
                 <update_rate>30.0</update_rate>
                 <camera>
-                    <horizontal_fov>${70.0*3.14/180.0}</horizontal_fov>
+                    <horizontal_fov>${70.0*PI/180.0}</horizontal_fov>
                     <image>
                         <width>512</width>
@@ -56,5 +57,5 @@
                 <update_rate>30.0</update_rate>
                 <camera name="${name}_camera">
-                    <horizontal_fov>${84.1*3.14/180.0}</horizontal_fov>
+                    <horizontal_fov>${84.1*PI/180.0}</horizontal_fov>
                     <image>
                         <width>1920</width>

File: kinect2_description/urdf/kinect2/kinect2-no-gazebo.xacro (robot description, xacro)
@@ -2,4 +2,5 @@
 <robot name="kinect2_sensor-ng" xmlns:xacro="http://www.ros.org/wiki/xacro">
     <xacro:macro name="kinect2_sensor-ng" params="name parent cam_px cam_py cam_pz cam_or cam_op cam_oy">
+    <xacro:property name="PI" value="3.14159265359" />
         <link name="${name}_link">
             <visual>
@@ -7,5 +8,5 @@
                     <mesh filename="package://kinect2_description/meshes/sensors/kinect2.dae"/>
                 </geometry>
-                <origin xyz="0.02 0 0" rpy="0 0 3.141592"/>
+                <origin xyz="0.02 0 0" rpy="0 0 ${PI}"/>
             </visual>
             <collision>
@@ -30,5 +31,5 @@
             <parent link="${name}_link"/>
             <child link="${name}_rgb_optical_frame"/>
-            <origin xyz="0 0.0125 0.016" rpy="-1.57 0 -1.57"/>
+            <origin xyz="0 0.0125 0.016" rpy="${-PI/2} 0 ${-PI/2}"/>
         </joint>
         <link name="${name}_depth_optical_frame"/>
@@ -36,5 +37,5 @@
             <parent link="${name}_link"/>
             <child link="${name}_depth_optical_frame"/>
-            <origin xyz="0 -0.0125 0.016" rpy="-1.57 0 -1.57"/>
+            <origin xyz="0 -0.0125 0.016" rpy="${-PI/2} 0 ${-PI/2}"/>
         </joint>
     </xacro:macro>
